File: InterfaceBoard/kicad/InterfaceBoard/InterfaceBoard.kicad_sch (KiCad schematic)
At the start: 48 parts, among them J1 MIDI IN, J10 JST Portamento Pot, J3 JST MIDI IN, J4 AudioJack2, J5 JST MIDI THRU, J6 JST GATE IN, J7 JST GATE CTRL, J8 JST Pitch Adj., J9 JST PWR, Q1 2N7000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

Commit message: Interface Board: Kicad: Minor fixes regarding JST connector orientation
Signed-off-by: CTXz <ctx.xda@gmail.com>
Parts:
- Q1, Q2, Q3, Q4: footprint Package_TO_SOT_THT:TO-92_Inline -> Package_TO_SOT_THT:TO-92_HandSolder
